Commit message: Fix end effector offset

File: nextagea_description/urdf/NextageAOpen.urdf (robot description, URDF)
Before this commit: robot NextageAOpen, 22 links, 21 joints
Joints:
- joint LARM_JOINT6: origin xyz=0 0 0 rpy=0 0 0 -> xyz=0 0 0.115 rpy=0 0 0
- joint RARM_JOINT6: origin xyz=0 0 0 rpy=0 0 0 -> xyz=0 0 0.115 rpy=0 0 0

Commit message: Add extra link for finger

File: nextagea_description/urdf/NextageAOpen.urdf (robot description, URDF)
Before this commit: robot NextageAOpen, 22 links, 21 joints
Links:
- added link LEND_EFFECTOR_finger
- added link REND_EFFECTOR_finger
Joints:
- added joint LARM_JOINT7: type fixed, parent LEND_EFFECTOR, child LEND_EFFECTOR_finger, origin xyz=0 0 0.115 rpy=0 0 0
- added joint RARM_JOINT7: type fixed, parent REND_EFFECTOR, child REND_EFFECTOR_finger, origin xyz=0 0 0.115 rpy=0 0 0
- joint LARM_JOINT6: origin xyz=0 0 0.115 rpy=0 0 0 -> xyz=0 0 0 rpy=0 0 0
- joint RARM_JOINT6: origin xyz=0 0 0.115 rpy=0 0 0 -> xyz=0 0 0 rpy=0 0 0

Commit message: Update with new end-effector

File: nextagea_description/urdf/NextageAOpen.urdf (robot description, URDF)
Before this commit: robot NextageAOpen, 24 links, 23 joints
Links:
- link LEND_EFFECTOR: geometry collision cylinder length=0.04 radius=0.035; visual cylinder length=0.04 radius=0.035
- link LEND_EFFECTOR_finger: geometry collision sphere radius=0.0125
- link REND_EFFECTOR: geometry collision cylinder length=0.04 radius=0.035; visual cylinder length=0.04 radius=0.035
- link REND_EFFECTOR_finger: geometry collision sphere radius=0.0125
Joints:
- joint LARM_JOINT7: origin xyz=0 0 0.115 rpy=0 0 0 -> xyz=-0.02 0 -0.115 rpy=0 0 0
- joint RARM_JOINT7: origin xyz=0 0 0.115 rpy=0 0 0 -> xyz=-0.02 0 -0.115 rpy=0 0 0
