Commit message: Fix the left arm

File: nextagea_description/urdf/NextageA_robot.xacro (robot description, xacro)
@@ -457,5 +457,5 @@
   </link>
   <xacro:transmission_nx_joint name="CHEST_JOINT0" />
-  <joint name="CHEST_JOINT0" type="revolute">
+  <joint name="CHEST_JOINT0" type="fixed">
     <parent link="WAIST"/>
     <child link="CHEST_JOINT0_Link"/>
@@ -466,5 +466,5 @@
   </joint>
   <xacro:transmission_nx_joint name="HEAD_JOINT0" />
-  <joint name="HEAD_JOINT0" type="revolute">
+  <joint name="HEAD_JOINT0" type="fixed">
     <parent link="CHEST_JOINT0_Link"/>
     <child link="HEAD_JOINT0_Link"/>
@@ -474,5 +474,5 @@
   </joint>
   <xacro:transmission_nx_joint name="HEAD_JOINT1" />
-  <joint name="HEAD_JOINT1" type="revolute">
+  <joint name="HEAD_JOINT1" type="fixed">
     <parent link="HEAD_JOINT0_Link"/>
     <child link="HEAD_JOINT1_Link"/>
@@ -482,5 +482,5 @@
   </joint>
   <xacro:transmission_nx_joint name="LARM_JOINT0" />
-  <joint name="LARM_JOINT0" type="revolute">
+  <joint name="LARM_JOINT0" type="fixed">
     <parent link="CHEST_JOINT0_Link"/>
     <child link="LARM_JOINT0_Link"/>
@@ -491,5 +491,5 @@
   </joint>
   <xacro:transmission_nx_joint name="LARM_JOINT1" />
-  <joint name="LARM_JOINT1" type="revolute">
+  <joint name="LARM_JOINT1" type="fixed">
     <parent link="LARM_JOINT0_Link"/>
     <child link="LARM_JOINT1_Link"/>
@@ -500,5 +500,5 @@
   </joint>
   <xacro:transmission_nx_joint name="LARM_JOINT2" />
-  <joint name="LARM_JOINT2" type="revolute">
+  <joint name="LARM_JOINT2" type="fixed">
     <parent link="LARM_JOINT1_Link"/>
     <child link="LARM_JOINT2_Link"/>
@@ -509,5 +509,5 @@
   </joint>
   <xacro:transmission_nx_joint name="LARM_JOINT3" />
-  <joint name="LARM_JOINT3" type="revolute">
+  <joint name="LARM_JOINT3" type="fixed">
     <parent link="LARM_JOINT2_Link"/>
     <child link="LARM_JOINT3_Link"/>
@@ -518,5 +518,5 @@
   </joint>
   <xacro:transmission_nx_joint name="LARM_JOINT4" />
-  <joint name="LARM_JOINT4" type="revolute">
+  <joint name="LARM_JOINT4" type="fixed">
     <parent link="LARM_JOINT3_Link"/>
     <child link="LARM_JOINT4_Link"/>
@@ -527,5 +527,5 @@
   </joint>
   <xacro:transmission_nx_joint name="LARM_JOINT5" />
-  <joint name="LARM_JOINT5" type="revolute">
+  <joint name="LARM_JOINT5" type="fixed">
     <parent link="LARM_JOINT4_Link"/>
     <child link="LARM_JOINT5_Link"/>
