Commit message: Edits for the fixed base

File: nextagea_description/urdf/NextageAOpen.urdf.xacro (robot description, xacro)
@@ -20,5 +20,5 @@
   <xacro:include filename="$(find nextagea_description)/urdf/nxao_gz_camera.xacro" />
   <xacro:arg name="fixed_base" default="true" />
-  <xacro:arg name="use_hand_cameras" default="false"/>
+  <xacro:arg name="use_hand_cameras" default="true"/>
   <xacro:arg name="use_ft_sensors" default="false"/>
   <xacro:arg name="use_cables_right" default="false"/>
@@ -99,9 +99,9 @@
       </collision>
       <!-- TODO: The inertial values are copied from ARM_JOINT5_Link. Replace with proper values. -->
-      <inertial>
-        <mass value="1.05156" />
+      <!-- <inertial>
+        <mass value="0.01" />
         <origin xyz="0.0 0.0 -0.08" rpy="0 -0 0"/>
         <inertia ixx="0.00194072" ixy="1.1e-07" ixz="-0.00042482" iyy="0.00209392" iyz="1.2e-07" izz="0.00035788"/>
-      </inertial>
+      </inertial> -->
     </link>
     <joint name="${prefix}ARM_ft_joint" type="fixed">
@@ -189,5 +189,5 @@
         <origin xyz="0 0.08 -0.1" rpy="0 0 0"/>
         <geometry>
-          <sphere radius="0.1"/>
+          <sphere radius="0.01"/>
         </geometry>
       </collision>
@@ -210,5 +210,5 @@
         <origin xyz="0 -0.08 -0.1" rpy="0 0 0"/>
         <geometry>
-          <sphere radius="0.1"/>
+          <sphere radius="0.01"/>
         </geometry>
       </collision>

File: nextagea_description/urdf/nxao_gz_camera.xacro (robot description, xacro)
@@ -37,5 +37,5 @@
 				<update_rate>30.0</update_rate>
 				<camera name="${camera_name}">
-					<horizontal_fov>1.3962634</horizontal_fov>
+					<horizontal_fov>2.3962634</horizontal_fov>
 					<image>
 						<width>800</width>
