Commit message: Add rotated extra link

File: nextage_description/urdf/general/common.xacro (robot description, xacro)
@@ -77,4 +77,10 @@
             </inertial>
             </link>
+            <link name="${camera_name}_color_frame"/>
+            <joint name="${camera_name}_color_joint" type="fixed">
+                <origin xyz="0 0 0" rpy="${-M_PI/2} 0 ${-M_PI/2}" />
+                <parent link="${camera_name}_Link" />
+                <child link="${camera_name}_color_frame" />
+            </joint>
             <gazebo reference="${camera_name}_Link">
                 <sensor type="camera" name="${camera_name}">

Commit message: Improved head cameras frame structure, added more accurate default values. Ready to add actual camera calibration data for each robot for best accuracy.

File: nextage_description/urdf/general/common.xacro (robot description, xacro)
@@ -41,5 +41,5 @@
         <!-- Properties -->
         <xacro:property name="M_PI" value="3.1415926535897931" />
-        <xacro:property name="jnt_head_camera_displacement_x" value="0.0175" />
+        <!-- <xacro:property name="jnt_head_camera_displacement_x" value="0.0175" />
         <xacro:property name="jnt_head_camera_displacement_y" value="0.0725" />
         <xacro:property name="jnt_head_camera_displacement_z" value="0.105" />
@@ -50,5 +50,5 @@
         <xacro:property name="jnt_hand_camera_displacement_z" value="0.0" />
         <xacro:property name="jnt_hand_camera_rot_y" value="1.5708" />
-        <xacro:property name="link_hand_camera_rot_z" value="0.0" />
+        <xacro:property name="link_hand_camera_rot_z" value="0.0" /> -->
         <xacro:macro name="camera_joint_link_gzplugin"
         params="camera_name link_parent jnt_displacement_x jnt_displacement_y jnt_displacement_z jnt_rotation_x jnt_rotation_y jnt_rotation_z link_displacement_x link_displacement_y link_displacement_z link_rotation_x link_rotation_y link_rotation_z">
@@ -123,4 +123,72 @@
             </gazebo>
         </xacro:macro>
+        <xacro:macro name="camera_joint_link_gzplugin2"
+        params="camera_name link_parent joint_xyz joint_rpy visual_xyz:='0 0 0.02' visual_rpy:='0 0 0'">
+            <joint name="${camera_name}" type="fixed">
+                <origin xyz="${joint_xyz}" rpy="${joint_rpy}" />
+                <parent link="${link_parent}" />
+                <child link="${camera_name}_Link" />
+            </joint>
+            <link name="${camera_name}_Link">
+                <visual>
+                    <origin xyz="${visual_xyz}" rpy="${visual_rpy}" />
+                    <geometry>
+                    <cylinder length="0.01" radius="0.015" />
+                    </geometry>
+                    <material name="Blue" />
+                </visual>
+                <inertial>
+                    <origin xyz="0 0 0" rpy="0 0 0" />
+                    <mass value="1e-6" />
+                    <inertia ixx="1e-12" ixy="0.0" ixz="0.0" iyy="1e-12" iyz="0.0"
+                    izz="1e-12" />
+                </inertial>
+            </link>
+            <!-- <link name="${camera_name}_color_frame"/>
+            <joint name="${camera_name}_color_joint" type="fixed">
+                <origin xyz="0 0 0" rpy="${-M_PI/2} 0 ${-M_PI/2}" />
+                <parent link="${camera_name}_Link" />
+                <child link="${camera_name}_color_frame" />
+            </joint> -->
+            <gazebo reference="${camera_name}_Link">
+                <sensor type="camera" name="${camera_name}">
+                    <update_rate>30.0</update_rate>
+                    <camera name="${camera_name}">
+                    <horizontal_fov>1.3962634</horizontal_fov>
+                    <image>
+                        <width>800</width>
+                        <height>800</height>
+                        <format>R8G8B8</format>
+                    </image>
+                    <clip>
+                        <near>0.1</near>
+                        <far>30</far>
+                    </clip>
+                    <noise>
+                        <type>gaussian</type>
+                        <!-- Noise is sampled independently per pixel on each frame. That pixel's
+                        noise value is added to each of its color channels, which at that point lie
+                        in the range [0,1]. -->
+                        <mean>0.0</mean>
+                        <stddev>0.007</stddev>
+                    </noise>
+                    </camera>
+                    <plugin name="camera_controller" filename="libgazebo_ros_camera.so">
+                    <alwaysOn>true</alwaysOn>
+                    <updateRate>0.0</updateRate>
+                    <cameraName>${camera_name}</cameraName>
+                    <imageTopicName>image_raw</imageTopicName>
+                    <cameraInfoTopicName>camera_info</cameraInfoTopicName>
+                    <frameName>${camera_name}_Link_frame</frameName>
+                    <hackBaseline>0.07</hackBaseline>
+                    <distortionK1>0.0</distortionK1>
+                    <distortionK2>0.0</distortionK2>
+                    <distortionK3>0.0</distortionK3>
+                    <distortionT1>0.0</distortionT1>
+                    <distortionT2>0.0</distortionT2>
+                    </plugin>
+                </sensor>
+            </gazebo>
+        </xacro:macro>
     </xacro:if>
     <xacro:macro name="sphere_inertia_def" params="radius mass">

File: nextage_description/urdf/robot/nextage_robot.xacro (robot description, xacro)
@@ -3,9 +3,10 @@
   <xacro:include filename="$(find nextage_description)/urdf/general/common.xacro" />
   <xacro:include filename="$(find nextage_description)/urdf/general/materials.xacro" />
+  <xacro:include filename="$(find nextage_description)/urdf/robot/NXA_default.xacro" />
   <xacro:macro name="nextage_robot" params="namespace:=/nextage/ nextage_gazebo_ros_control:=true">
     <!-- NOTE: The poses of headmount and hand cameras are NOT precisely adjusted to
     the 3D model nor the actual hardware config. These configs
     are meant for a rapid prototyping only. -->
-    <xacro:camera_joint_link_gzplugin
+    <!-- <xacro:camera_joint_link_gzplugin
         camera_name="CAMERA_HEAD_L" link_parent="HEAD_JOINT1_Link"
         jnt_displacement_x="${jnt_head_camera_displacement_x}" jnt_displacement_y="${jnt_head_camera_displacement_y}" jnt_displacement_z="${jnt_head_camera_displacement_z}"
@@ -18,5 +19,13 @@
         jnt_rotation_x="0" jnt_rotation_y="${radians(15)}" jnt_rotation_z="${radians(5)}"
         link_displacement_x="0.0325" link_displacement_y="0" link_displacement_z="0"
-        link_rotation_x="0" link_rotation_y="${M_PI/2}" link_rotation_z="${link_head_camera_rot_z}" />
+        link_rotation_x="0" link_rotation_y="${M_PI/2}" link_rotation_z="${link_head_camera_rot_z}" /> -->
+    <xacro:camera_joint_link_gzplugin2
+        camera_name="CAMERA_HEAD_L" link_parent="HEAD_JOINT1_Link"
+        joint_xyz="${jnt_head_to_leye_xyz}"
+        joint_rpy="${jnt_head_to_leye_rpy}" />
+    <xacro:camera_joint_link_gzplugin2
+        camera_name="CAMERA_HEAD_R" link_parent="CAMERA_HEAD_L_Link"
+        joint_xyz="${jnt_leye_to_reye_xyz}"
+        joint_rpy="${jnt_leye_to_reye_rpy}" />
     <xacro:gazebo_nx_link name="WAIST" color="Black" />
     <link name="WAIST">
